Commit message: Mobile Boat Update

File: urdf/WATER.xacro (robot description, xacro)
@@ -8,5 +8,5 @@
   <inertial>
     <origin rpy="0 0 0" xyz="0.041985844365174226 0.5041551418509241 0.11753492516942377"/>
-    <mass value="731.907802985047"/>
+    <mass value="91"/>
     <inertia ixx="102.253408" ixy="0.944947" ixz="0.571694" iyy="75.226668" iyz="0.019964" izz="175.055626"/>
   </inertial>
@@ -70,12 +70,33 @@
 <link name="propeller_left_1">
   <inertial>
-    <origin rpy="0 0 0" xyz="-0.02469707240420338 8.693535857862145e-08 3.533814449951933e-07"/>
-    <mass value="0.4577791370132495"/>
-    <inertia ixx="0.00083" ixy="0.0" ixz="-0.0" iyy="0.000457" iyz="-0.0" izz="0.000457"/>
+    <origin rpy="0 0 0" xyz="-0.02465138415626883 -3.202893716913735e-07 -5.662137425588298e-15"/>
+    <mass value="0.861936288291951"/>
+    <inertia ixx="0.001968" ixy="-0.0" ixz="0.0" iyy="0.001151" iyz="-0.0" izz="0.001151"/>
+  </inertial>
+  <visual>
+    <origin rpy="0 0 0" xyz="0.497574 -0.206555 -0.715"/>
+    <geometry>
+      <mesh filename="package://WATER_description/meshes/propeller_left_1.stl" scale="0.001 0.001 0.001"/>
+    </geometry>
+    <material name="silver"/>
+  </visual>
+  <collision>
+    <origin rpy="0 0 0" xyz="0.497574 -0.206555 -0.715"/>
+    <geometry>
+      <mesh filename="package://WATER_description/meshes/propeller_left_1.stl" scale="0.001 0.001 0.001"/>
+    </geometry>
+  </collision>
+</link>
+<!--Right Propeller-->
+<link name="propeller_left_3">
+  <inertial>
+    <origin rpy="0 0 0" xyz="-0.024651081039449574 8.693535802350993e-08 3.5338152826192015e-07"/>
+    <mass value="0.861936288291951"/>
+    <inertia ixx="0.001968" ixy="0.0" ixz="0.0" iyy="0.001151" iyz="-0.0" izz="0.001151"/>
   </inertial>
   <visual>
     <origin rpy="0 0 0" xyz="0.521155 -0.767824 -0.713099"/>
     <geometry>
-      <mesh filename="package://WATER_description/meshes/propeller_left_1.stl" scale="0.001 0.001 0.001"/>
+      <mesh filename="package://WATER_description/meshes/propeller_left_3.stl" scale="0.001 0.001 0.001"/>
     </geometry>
     <material name="silver"/>
@@ -84,26 +105,5 @@
     <origin rpy="0 0 0" xyz="0.521155 -0.767824 -0.713099"/>
     <geometry>
-      <mesh filename="package://WATER_description/meshes/propeller_left_1.stl" scale="0.001 0.001 0.001"/>
-    </geometry>
-  </collision>
-</link>
-<!--Right Propeller-->
-<link name="propeller_right_1">
-  <inertial>
-    <origin rpy="0 0 0" xyz="-0.024697375521022857 -3.2028937094197296e-07 -8.881784197001252e-14"/>
-    <mass value="0.4577791370132495"/>
-    <inertia ixx="0.00083" ixy="-0.0" ixz="-0.0" iyy="0.000457" iyz="-0.0" izz="0.000457"/>
-  </inertial>
-  <visual>
-    <origin rpy="0 0 0" xyz="0.497574 -0.206555 -0.715"/>
-    <geometry>
-      <mesh filename="package://WATER_description/meshes/propeller_right_1.stl" scale="0.001 0.001 0.001"/>
-    </geometry>
-    <material name="silver"/>
-  </visual>
-  <collision>
-    <origin rpy="0 0 0" xyz="0.497574 -0.206555 -0.715"/>
-    <geometry>
-      <mesh filename="package://WATER_description/meshes/propeller_right_1.stl" scale="0.001 0.001 0.001"/>
+      <mesh filename="package://WATER_description/meshes/propeller_left_3.stl" scale="0.001 0.001 0.001"/>
     </geometry>
   </collision>
@@ -148,5 +148,5 @@
   <child link="propeller_left_1"/>
   <axis xyz="-1.0 0.0 0.0"/>
-  <limit effort="50" velocity="1"/>
+  <limit effort="300" velocity="10"/>
 </joint>
 <!--Right Propller Joint-->
@@ -154,7 +154,7 @@
   <origin rpy="0 0 0" xyz="-0.060785 0.0 0.525"/>
   <parent link="motor_support_right_1"/>
-  <child link="propeller_right_1"/>
+  <child link="propeller_left_3"/>
   <axis xyz="-1.0 0.0 -0.0"/>
-  <limit effort="50" velocity="1"/>
+  <limit effort="300" velocity="10"/>
 </joint>
 <!--Camera Joint-->
@@ -164,4 +164,26 @@
   <child link="camera_link_1"/>
 </joint>
+<!--Tranmission for Right Propller-->
+<transmission name="simple_trans_right">
+  <type>transmission_interface/SimpleTransmission</type>
+  <joint name="Rev19">
+    <hardwareInterface>VelocityJointInterface</hardwareInterface>
+  </joint>
+  <actuator name="Right_propeller_motor">
+    <mechanicalReduction>1</mechanicalReduction>
+    <hardwareInterface>VelocityJointInterface</hardwareInterface>
+  </actuator>
+</transmission>
+<!--Tranmission for Left Propller-->
+<transmission name="simple_trans_left">
+  <type>transmission_interface/SimpleTransmission</type>
+  <joint name="Rev18">
+    <hardwareInterface>VelocityJointInterface</hardwareInterface>
+  </joint>
+  <actuator name="Left_propeller_motor">
+    <mechanicalReduction>1</mechanicalReduction>
+    <hardwareInterface>VelocityJointInterface</hardwareInterface>
+  </actuator>
+</transmission>
 <!--Camera Plugin-->
   <gazebo reference="camera_link_1">

Commit message: Mobile Boat Update

File: urdf/WATER.xacro (robot description, xacro)
@@ -2,5 +2,5 @@
 <robot name="WATER" xmlns:xacro="http://www.ros.org/wiki/xacro">
 <xacro:include filename="$(find WATER_description)/urdf/materials.xacro" />
-<xacro:include filename="$(find WATER_description)/urdf/WATER.trans" />
+<!--<xacro:include filename="$(find WATER_description)/urdf/WATER.trans" />-->
 <xacro:include filename="$(find WATER_description)/urdf/WATER.gazebo" />
 <!--Base Link/ Boat Hull-->
@@ -8,5 +8,5 @@
   <inertial>
     <origin rpy="0 0 0" xyz="0.041985844365174226 0.5041551418509241 0.11753492516942377"/>
-    <mass value="91"/>
+    <mass value="100.05"/>
     <inertia ixx="102.253408" ixy="0.944947" ixz="0.571694" iyy="75.226668" iyz="0.019964" izz="175.055626"/>
   </inertial>
@@ -29,5 +29,5 @@
   <inertial>
     <origin rpy="0 0 0" xyz="-0.00038428463028200577 -1.931763642015749e-05 0.2794011308123638"/>
-    <mass value="10.796675596228138"/>
+    <mass value="1"/>
     <inertia ixx="0.281164" ixy="-2.4e-05" ixz="0.002165" iyy="0.281586" iyz="-0.0003" izz="0.004869"/>
   </inertial>
@@ -50,5 +50,5 @@
   <inertial>
     <origin rpy="0 0 0" xyz="-0.005187497162707055 0.13542109450750728 0.37290152359449974"/>
-    <mass value="20.721819356800275"/>
+    <mass value="1"/>
     <inertia ixx="1.104335" ixy="0.022331" ixz="0.012255" iyy="0.483329" iyz="-0.286828" izz="0.631875"/>
   </inertial>
@@ -71,5 +71,5 @@
   <inertial>
     <origin rpy="0 0 0" xyz="-0.02465138415626883 -3.202893716913735e-07 -5.662137425588298e-15"/>
-    <mass value="0.861936288291951"/>
+    <mass value="0.025"/>
     <inertia ixx="0.001968" ixy="-0.0" ixz="0.0" iyy="0.001151" iyz="-0.0" izz="0.001151"/>
   </inertial>
@@ -92,5 +92,5 @@
   <inertial>
     <origin rpy="0 0 0" xyz="-0.024651081039449574 8.693535802350993e-08 3.5338152826192015e-07"/>
-    <mass value="0.861936288291951"/>
+    <mass value="0.025"/>
     <inertia ixx="0.001968" ixy="0.0" ixz="0.0" iyy="0.001151" iyz="-0.0" izz="0.001151"/>
   </inertial>
@@ -113,5 +113,5 @@
   <inertial>
     <origin rpy="0 0 0" xyz="3.962738093221674e-08 -1.2711576602431052e-07 0.025000000000001354"/>
-    <mass value="7.85"/>
+    <mass value="0.05"/>
     <inertia ixx="0.027778" ixy="0.000684" ixz="-0.0" iyy="0.008201" iyz="0.0" izz="0.032708"/>
   </inertial>
@@ -127,4 +127,25 @@
     <geometry>
       <mesh filename="package://WATER_description/meshes/camera_link_1.stl" scale="0.001 0.001 0.001"/>
+    </geometry>
+  </collision>
+</link>
+<!--Balance Link-->
+<link name="balance_1">
+  <inertial>
+    <origin rpy="0 0 0" xyz="0.024984655377752518 0.0008720125959205127 0.049999999999999184"/>
+    <mass value="2.1"/>
+    <inertia ixx="0.059224" ixy="0.001711" ixz="0.0" iyy="0.010281" iyz="-0.0" izz="0.053151"/>
+  </inertial>
+  <visual>
+    <origin rpy="0 0 0" xyz="-0.332254 -0.514292 -0.19"/>
+    <geometry>
+      <mesh filename="package://WATER_description/meshes/balance_1.stl" scale="0.001 0.001 0.001"/>
+    </geometry>
+    <material name="silver"/>
+  </visual>
+  <collision>
+    <origin rpy="0 0 0" xyz="-0.332254 -0.514292 -0.19"/>
+    <geometry>
+      <mesh filename="package://WATER_description/meshes/balance_1.stl" scale="0.001 0.001 0.001"/>
     </geometry>
   </collision>
@@ -164,13 +185,18 @@
   <child link="camera_link_1"/>
 </joint>
+<joint name="Rigid21" type="fixed">
+  <origin rpy="0 0 0" xyz="0.332254 0.514292 0.19"/>
+  <parent link="base_link"/>
+  <child link="balance_1"/>
+</joint>
 <!--Tranmission for Right Propller-->
 <transmission name="simple_trans_right">
   <type>transmission_interface/SimpleTransmission</type>
   <joint name="Rev19">
-    <hardwareInterface>VelocityJointInterface</hardwareInterface>
+    <hardwareInterface>hardware_interface/VelocityJointInterface</hardwareInterface>
   </joint>
   <actuator name="Right_propeller_motor">
     <mechanicalReduction>1</mechanicalReduction>
-    <hardwareInterface>VelocityJointInterface</hardwareInterface>
+    <hardwareInterface>hardware_interface/VelocityJointInterface</hardwareInterface>
   </actuator>
 </transmission>
@@ -179,47 +205,10 @@
   <type>transmission_interface/SimpleTransmission</type>
   <joint name="Rev18">
-    <hardwareInterface>VelocityJointInterface</hardwareInterface>
+    <hardwareInterface>hardware_interface/VelocityJointInterface</hardwareInterface>
   </joint>
   <actuator name="Left_propeller_motor">
     <mechanicalReduction>1</mechanicalReduction>
-    <hardwareInterface>VelocityJointInterface</hardwareInterface>
+    <hardwareInterface>hardware_interface/VelocityJointInterface</hardwareInterface>
   </actuator>
 </transmission>
-<!--Camera Plugin-->
-  <gazebo reference="camera_link_1">
-    <sensor type="camera" name="camera1">
-      <update_rate>30.0</update_rate>
-      <camera name="head">
-        <horizontal_fov>1.3962634</horizontal_fov>
-        <image>
-          <width>800</width>
-          <height>800</height>
-          <format>R8G8B8</format>
-        </image>
-        <clip>
-          <near>0.02</near>
-          <far>300</far>
-        </clip>
-        <noise>
-          <type>gaussian</type>
-          <mean>0.0</mean>
-          <stddev>0.007</stddev>
-        </noise>
-      </camera>
-      <plugin name="camera_controller" filename="libgazebo_ros_camera.so">
-        <alwaysOn>true</alwaysOn>
-        <updateRate>0.0</updateRate>
-        <cameraName>rrbot/camera1</cameraName>
-        <imageTopicName>image_raw</imageTopicName>
-        <cameraInfoTopicName>camera_info</cameraInfoTopicName>
-        <frameName>camera_link</frameName>
-        <hackBaseline>0.07</hackBaseline>
-        <distortionK1>0.0</distortionK1>
-        <distortionK2>0.0</distortionK2>
-        <distortionK3>0.0</distortionK3>
-        <distortionT1>0.0</distortionT1>
-        <distortionT2>0.0</distortionT2>
-      </plugin>
-    </sensor>
-  </gazebo>
 </robot>
